File: hardware/kicad/frontpanel/frontpanel.kicad_pcb (KiCad board)
At the start: 2 copper layers, 120 x 136 mm, 47 parts, among them J14 Fader 1 (MOT+ MOT- GND 3V3 WI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, J15 Fader 2 (MOT+ MOT- GND 3V3 WI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, J16 Fader 3 (MOT+ MOT- GND 3V3 WI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, J17 Fader 4 (MOT+ MOT- GND 3V3 WI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, J9 IDC 2x15 <- Mainboard, Q1 BC327, Q2 BC337, SW1 Soft-Key 1, SW10 Makro 4, SW2 Soft-Key 2, SW3 Soft-Key 3, SW4 Soft-Key 4, SW5 Soft-Key 5, SW6 Soft-Key 6, SW7 Makro 1, SW8 Makro 2, SW9 Makro 3, U8 MCP23017-E/SP, U9 MPR121 Breakout

Commit message: Session 2026-10-03 00:27: Reserve raus (Stepper, C3, GPIO45, 7 Loetjumper), alle drei Platinen neu geroutet; Push und Falle 18 behoben
Parts:
- removed JP10: INTB->IO_INT, SolderJumper-2_P1.3mm_Open_RoundedPad1.0x1.5mm
- removed JP11: BL: 1=MCP 3=GPIO45, SolderJumper-3_P1.3mm_Bridged12_RoundedPad1.0x1.5mm_NumberLabels
- removed JP9: INTA->IO_INT, SolderJumper-2_P1.3mm_Bridged_RoundedPad1.0x1.5mm
- removed Q2: BC337, TO-92_Inline
- removed R12: 100k, R_Axial_DIN0207_L6.3mm_D2.5mm_P10.16mm_Horizontal
- removed R9: 1k, R_Axial_DIN0207_L6.3mm_D2.5mm_P10.16mm_Horizontal
- added R17: 10k, R_Axial_DIN0207_L6.3mm_D2.5mm_P10.16mm_Horizontal, F.Cu at (24.9, 86.0)
Connections:
- J9 pad 29: BELLY_BL_PWM -> DISP_RST
- R11 pad 1: BL_Q2C -> BL_EN_MCP
- U8 pad 19: INTB -> (no net)
- U8 pad 20: INTA -> IO_INT
Routing:
- net BELLY_BL_PWM: track 131.0 -> 0.00 mm, vias 1 -> 0
- net DISP_RST: track 89.4 -> 182.8 mm, vias 1 -> 2
- net GND: track 613.8 -> 571.1 mm
- net FADER2_WIPER: track 164.5 -> 126.3 mm, vias 2 -> 1
- net BL_EN_MCP: track 91.1 -> 123.1 mm, vias 2 -> 3
- net FADER1_WIPER: track 134.1 -> 164.1 mm
- net KEY10: track 74.9 -> 102.0 mm
- net I2C_SCL: track 136.1 -> 111.1 mm, vias 0 -> 1
- net INTA: track 23.9 -> 0.00 mm, vias 1 -> 0
- net INTB: track 21.5 -> 0.00 mm, vias 1 -> 0
- net BL_DRV: track 21.3 -> 0.00 mm
- net MOT2B: track 109.3 -> 88.1 mm
- net BL_Q2C: track 20.4 -> 0.00 mm
- net ENC_A: track 109.8 -> 128.5 mm, vias 0 -> 2
- net IO_INT: track 131.5 -> 113.2 mm
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
Commit message: Session 2026-10-09 11:37: Platinen finalisiert: Teile von Reichelt, Silkscreen mit Logo und Pin-Namen, alle drei Boards neu geroutet
Parts:
- removed U9: MPR121 Breakout, MPR121_Breakout
- added J18: MPR121 per Kabel (ADDR am Modul an GND), PinHeader_1x09_P2.54mm_Vertical, F.Cu at (81.8, 88.0)
- moved R17 37.5 mm to (12.9, 121.5)
Routing:
- net FADER1_WIPER: track 164.1 -> 131.4 mm
- net TOUCH2: track 49.1 -> 20.5 mm
- net MOT1B: track 93.9 -> 69.2 mm, vias 3 -> 0
- net I2C_SCL: track 111.1 -> 134.4 mm, vias 1 -> 0
- net 3V3: track 394.9 -> 371.9 mm
- net KEY10: track 102.0 -> 79.1 mm, vias 1 -> 0
- net I2C_SDA: track 112.4 -> 132.1 mm
- net ENC_A: track 128.5 -> 109.9 mm, vias 2 -> 0
- net TOUCH4: track 50.6 -> 33.3 mm, vias 0 -> 1
- net FADER3_WIPER: track 133.7 -> 117.5 mm
- net SPI_MOSI: track 144.7 -> 129.0 mm, vias 3 -> 0
- net MOT2A: track 116.4 -> 130.9 mm, vias 1 -> 5
- net BL_EN_MCP: track 123.1 -> 137.4 mm, vias 3 -> 1
- net MOT3B: track 73.2 -> 59.0 mm
- net TOUCH1: track 84.9 -> 98.8 mm
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Other:
- board text added: "3V3"
- board text added: "CS"
- board text added: "DC"
- board text added: "DESK-MATE"
- board text added: "DESK-MATE · FRONTPANEL · Rev 1"
- board text added: "DISPLAY 2,8 ZOLL"
- board text added: "FADER 1"
- board text added: "FADER 2"
- board text added: "FADER 3"
- board text added: "FADER 4"
- board text added: "FRONTPANEL · DECK"
- board text added: "Frontpanel Rev 1"
- board text added: "GND"
- board text added: "IRQ"
- board text added: "JLCJLCJLCJLC"
- board text added: "LED"
- board text added: "Leon Fröhlich · 2026"
- board text added: "M+"
- board text added: "M-"
- board text added: "MAINBOARD"
- board text added: "MPR121"
- board text added: "RST"
- board text added: "Rev 1 · 2026-10"
- board text added: "SCK"
- board text added: "SCL"
- board text added: "SDA"
- board text added: "SDI"
- board text added: "SDO"
- board text added: "T1"
- board text added: "T2"
- board text added: "T3"
- board text added: "T4"
- board text added: "TCH"
- board text added: "T_CLK"
- board text added: "T_CS"
- board text added: "T_DIN"
- board text added: "T_DO"
- board text added: "T_IRQ"
- board text added: "VCC"
- board text added: "WIP"
- board text removed: "Desk-Mate frontpanel v1 2026-08"
