File: hardware/kicad/frontpanel/frontpanel.kicad_sch (KiCad schematic)
At the start: 47 parts, among them J14 Fader 1 (MOT+ MOT- GND 3V3 WI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, J15 Fader 2 (MOT+ MOT- GND 3V3 WI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, J16 Fader 3 (MOT+ MOT- GND 3V3 WI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, J17 Fader 4 (MOT+ MOT- GND 3V3 WI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, J9 IDC 2x15 <- Mainboard, Q1 BC327, Q2 BC337, SW1 Soft-Key 1, SW10 Makro 4, SW2 Soft-Key 2, SW3 Soft-Key 3, SW4 Soft-Key 4, SW5 Soft-Key 5, SW6 Soft-Key 6, SW7 Makro 1, SW8 Makro 2, SW9 Makro 3, U8 MCP23017-E/SP, U9 MPR121 Breakout

Commit message: Session 2026-10-03 00:27: Reserve raus (Stepper, C3, GPIO45, 7 Loetjumper), alle drei Platinen neu geroutet; Push und Falle 18 behoben
Parts:
- removed JP10: INTB->IO_INT, Jumper:SolderJumper-2_P1.3mm_Open_RoundedPad1.0x1.5mm, symbol Jumper:SolderJumper_2_Open
- removed JP11: BL: 1=MCP 3=GPIO45, Jumper:SolderJumper-3_P1.3mm_Bridged12_RoundedPad1.0x1.5mm_NumberLabels, symbol Jumper:SolderJumper_3_Bridged12
- removed JP9: INTA->IO_INT, Jumper:SolderJumper-2_P1.3mm_Bridged_RoundedPad1.0x1.5mm, symbol Jumper:SolderJumper_2_Bridged
- removed Q2: BC337, Package_TO_SOT_THT:TO-92_Inline, symbol Transistor_BJT:BC337
- removed R12: 100k, Resistor_THT:R_Axial_DIN0207_L6.3mm_D2.5mm_P10.16mm_Horizontal, symbol Device:R
- removed R9: 1k, Resistor_THT:R_Axial_DIN0207_L6.3mm_D2.5mm_P10.16mm_Horizontal, symbol Device:R
- added R17: 10k, Resistor_THT:R_Axial_DIN0207_L6.3mm_D2.5mm_P10.16mm_Horizontal, symbol Device:R
Connections:
- net BELLY_BL_PWM is gone; now on net DISP_RST: J9.29 (Pin_29)
- net BL_Q2C is gone; now on net BL_EN_MCP: R11.1
- net INTA is gone; now on net IO_INT: U8.20 (INTA)
- net 3V3: now also R17.2
- net DISP_RST: now also R17.1
- net INTB: no longer names the net of U8.19 (INTB)
- no-connect marks 17 -> 18
Other:
- note added: "Bauch-Display ILI9341 2.8in SPI (MSP2807, 14-Pin, Header links); Backlight 150 mA: High-Side BC327 direkt vom MCP GPB6 (low = an); 10k B-E haelt aus, bis der MCP konfiguriert ist"
- note added: "MCP23017 (0x20): Tasten 1-10 gegen GND (interne Pull-ups), Encoder, DISP_RST (10k Pull-up, geht ueber IDC 29 auch zu den Augen), Backlight-Enable; INTA direkt an IO_INT"
- note removed: "Bauch-Display ILI9341 2.8in SPI (MSP2807, 14-Pin, Header links); Backlight 150 mA: High-Side BC327 via BC337, Quelle JP11 (1=MCP GPB6, 3=GPIO45-PWM)"
- note removed: "MCP23017 (0x20): Tasten 1-10 gegen GND (interne Pull-ups), Encoder, DISP_RST, Backlight-Enable; INTA -> IO_INT"
- moved on the sheet: C13, C14, ENC1, R10, R11, SW1, SW10, SW2, SW3, SW4, SW5, SW6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

Commit message: Session 2026-10-09 11:37: Platinen finalisiert: Teile von Reichelt, Silkscreen mit Logo und Pin-Namen, alle drei Boards neu geroutet
Parts:
- removed U9: MPR121 Breakout, deskmate:MPR121_Breakout, symbol deskmate:MPR121_Breakout
- added J18: MPR121 per Kabel (ADDR am Modul an GND), Connector_PinHeader_2.54mm:PinHeader_1x09_P2.54mm_Vertical, symbol Connector_Generic:Conn_01x09
Connections:
- net 3V3: now also J18.1 (Pin_1)
- net GND: now also J18.2 (Pin_2)
- net I2C_SCL: now also J18.3 (Pin_3)
- net I2C_SDA: now also J18.4 (Pin_4)
- net IO_INT: now also J18.5 (Pin_5)
- net TOUCH1: now also J18.6 (Pin_6)
- net TOUCH2: now also J18.7 (Pin_7)
- net TOUCH3: now also J18.8 (Pin_8)
- net TOUCH4: now also J18.9 (Pin_9)
- no-connect marks 18 -> 10
Other:
- note added: "Fader X32 (panel-mount, Draehte an Stiftleisten): Motor auf IDC, Schleifer ueber RC 1k/100n, Touch ueber J18 zum MPR121 (Modul per Kabel, kein Sockel: Clone-Raster unbelegt, Falle 15)"
- note removed: "Fader X32 (panel-mount, Draehte an Stiftleisten): Motor auf IDC, Schleifer ueber RC 1k/100n, Touch auf MPR121 ELE0-3"
- moved on the sheet: H10, H11, H12, H5, H6, H7, H8, H9
