File: hardware/kicad/mainboard/mainboard.kicad_pcb (KiCad board)
At the start: 2 copper layers, 100 x 100 mm, 50 parts, among them J1 USB-C 5V/3A (GCT USB4085), J10 Stepper 1A 1B 2A 2B, J2 IDC 2x15 -> Frontpanel, J3 Servo Pan (GND/5V/Sig), J4 Servo Tilt (GND/5V/Sig), J5 ARGB 5V/GND/Data, J6 BME680 (VCC GND SCL SDA SDO C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, J7 Augen-Kabel, J8 RST/BOOT extern, U1 ESP32-S3-DevKitC-1-N16R8, U2 LD1117V33, U3 DRV8833 Pololu #2130, U4 DRV8833 Pololu #2130 (Fader 3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, U5 MT3608 Boost ~9V (optional, 4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, U6 ESP32-C3 SuperMini Reserve, U7 A4988/TMC2209 Reserve

Commit message: Session 2026-08-31 12:22: Arbeitsstand
Parts:
- moved C7 76.6 mm to (134.5, 72.4)
- moved D1 76.6 mm to (103.4, 73.4)
- moved H1 76.6 mm to (58.0, 58.4)
- moved J1 76.6 mm to (106.0, 56.0)
- moved J10 76.6 mm to (100.2, 119.9)
- moved J3 76.6 mm to (148.5, 97.9)
- moved J4 76.6 mm to (148.5, 109.9)
- moved J5 76.6 mm to (148.5, 121.9)
- moved R5 76.6 mm to (143.0, 107.5)
- moved U2 76.6 mm to (124.5, 77.3)
- moved U5 76.6 mm to (132.0, 84.6)
- moved C1 76.6 mm to (124.5, 66.4)
- moved C11 76.6 mm to (135.7, 66.4)
- moved C2 76.6 mm to (105.7, 114.4)
- moved C3 76.6 mm to (121.7, 114.4)
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
Commit message: Session 2026-10-03 00:27: Reserve raus (Stepper, C3, GPIO45, 7 Loetjumper), alle drei Platinen neu geroutet; Push und Falle 18 behoben
Parts:
- removed C8: 100u, CP_Radial_D6.3mm_P2.50mm
- removed J10: Stepper 1A 1B 2A 2B, PinHeader_1x04_P2.54mm_Vertical
- removed JP2: C3 TX->S3 RX0, SolderJumper-2_P1.3mm_Open_RoundedPad1.0x1.5mm
- removed JP3: S3 TX0->C3 RX, SolderJumper-2_P1.3mm_Open_RoundedPad1.0x1.5mm
- removed JP4: VM: 1=5V 3=Boost, SolderJumper-3_P1.3mm_Bridged12_RoundedPad1.0x1.5mm_NumberLabels
- removed JP5: nSLEEP an 3V3, SolderJumper-2_P1.3mm_Bridged_RoundedPad1.0x1.5mm
- removed JP6: STEP<-FADER3_PWM, SolderJumper-2_P1.3mm_Open_RoundedPad1.0x1.5mm
- removed JP7: DIR<-FADER3_DIR, SolderJumper-2_P1.3mm_Open_RoundedPad1.0x1.5mm
- removed JP8: EN<-FADER4_PWM, SolderJumper-2_P1.3mm_Open_RoundedPad1.0x1.5mm
- removed U6: ESP32-C3 SuperMini Reserve, ESP32-C3_SuperMini
- removed U7: A4988/TMC2209 Reserve, A4988_Socket
- JP1: value BL45 (Strapping! offen lassen ausser Backlight-PWM) -> VM: 1=5V 3=Boost; footprint SolderJumper-2_P1.3mm_Open_RoundedPad1.0x1.5mm -> SolderJumper-3_P1.3mm_Bridged12_RoundedPad1.0x1.5mm_NumberLabels
- moved JP1 79.9 mm to (58.0, 31.0)
- moved C7 76.6 mm to (80.5, 18.0)
- moved D1 76.6 mm to (49.4, 19.0)
- moved H1 76.6 mm to (4.00, 4.00)
- moved J1 76.6 mm to (52.0, 1.57)
- moved J3 76.6 mm to (94.5, 43.5)
- moved J4 76.6 mm to (94.5, 55.5)
- moved J5 76.6 mm to (94.5, 67.5)
- moved R5 76.6 mm to (89.0, 53.1)
- moved U2 76.6 mm to (70.5, 22.9)
- moved U5 76.6 mm to (78.0, 30.2)
- moved C1 76.6 mm to (70.5, 12.0)
- moved C11 76.6 mm to (81.7, 12.0)
- moved C2 76.6 mm to (51.7, 60.0)
- moved C3 76.6 mm to (67.7, 60.0)
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Connections:
- J2 pad 29: BELLY_BL_PWM -> DISP_RST
- J7 pad 10: GND -> DISP_RST
- JP1 pad 1: BL_PWM_45 -> 5V
- JP1 pad 2: BELLY_BL_PWM -> VM
- U1 pad 24: UART0_TX -> (no net)
- U1 pad 25: UART0_RX -> (no net)
- U1 pad 37: BL_PWM_45 -> (no net)
- U3 pad 7: DRV_SLEEP -> 3V3
- U4 pad 7: DRV_SLEEP -> 3V3
Routing:
- net DISP_RST: track 0.00 -> 89.5 mm, vias 0 -> 1
- net BELLY_BL_PWM: track 78.0 -> 0.00 mm, vias 3 -> 0
- net WS2812_DATA: track 87.6 -> 153.4 mm, vias 1 -> 0
- net GND: track 528.2 -> 462.7 mm
- net UART0_RX: track 65.3 -> 0.00 mm
- net UART0_TX: track 63.2 -> 0.00 mm
- net FADER4_PWM: track 90.5 -> 39.6 mm, vias 2 -> 0
- net FADER3_DIR: track 93.5 -> 50.9 mm, vias 3 -> 1
- net DRV_SLEEP: track 38.5 -> 0.00 mm, vias 1 -> 0
- net STEP_EN: track 38.4 -> 0.00 mm
- net BL_PWM_45: track 37.6 -> 0.00 mm
- net C3_TX: track 34.7 -> 0.00 mm
- net STEP_STEP: track 29.7 -> 0.00 mm
- net STEP_DIR: track 29.5 -> 0.00 mm
- net SPI_DC: track 184.0 -> 155.9 mm, vias 0 -> 2
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
Commit message: Session 2026-10-09 11:37: Platinen finalisiert: Teile von Reichelt, Silkscreen mit Logo und Pin-Namen, alle drei Boards neu geroutet
Parts:
- C1: value 1000u/10V -> 1000u/16V
- C11: footprint CP_Radial_D5.0mm_P2.50mm -> CP_Radial_D5.0mm_P2.00mm
- J1: value USB-C 5V/3A (GCT USB4085) -> USB-C-Breakout 5V/3A (VBUS GND CC1 CC2); footprint USB_C_Receptacle_GCT_USB4085 -> TerminalBlock_Phoenix_MKDS-1,5-4-5.08_1x04_P5.08mm_Horizontal
- J3, J4, J5: footprint JST_XH_B3B-XH-A_1x03_P2.50mm_Vertical -> PinHeader_1x03_P2.54mm_Vertical
- J6: value BME680 (VCC GND SCL SDA SDO CS) -> I2C / BME680 per Kabel; footprint PinSocket_1x06_P2.54mm_Vertical -> PinHeader_1x04_P2.54mm_Vertical
- J7: value Augen-Kabel -> Augen-Kabel IDC 2x5; footprint PinHeader_1x10_P2.54mm_Vertical -> IDC-Header_2x05_P2.54mm_Vertical
- U1: value ESP32-S3-DevKitC-1-N16R8 -> ESP32-S3-DevKitC-1 (N16R8/N8R8)
- moved R1 12.1 mm to (34.9, 14.5), turned to 0 degrees
- moved J1 8.99 mm to (44.4, 6.30)
- moved J7 6.48 mm to (93.7, 16.4)
- moved J3 5.64 mm to (97.0, 38.5), turned to 0 degrees
- moved J4 5.64 mm to (97.0, 50.5), turned to 0 degrees
- moved J5 5.64 mm to (97.0, 62.5), turned to 0 degrees
- moved U5 3.05 mm to (75.2, 29.0), turned to 90 degrees
- moved J6 2.57 mm to (78.2, 3.60)
- moved D1 2.00 mm to (49.4, 21.0)
- moved F1 2.00 mm to (55.0, 15.5)
- moved C6 1.50 mm to (52.5, 26.5)
- moved R2 1.00 mm to (34.9, 18.5)
- moved R3 1.00 mm to (34.9, 22.5)
- moved R4 1.00 mm to (34.9, 26.5)
- moved TP1 1.00 mm to (65.0, 4.00)
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Connections:
- J7 pad 2: 3V3 -> GND
- J7 pad 3: GND -> SPI_SCK
- J7 pad 6: SPI_SCK -> GND
Routing:
- net WS2812_DATA: track 153.4 -> 89.2 mm
- net CS_EYE_L: track 106.3 -> 137.9 mm, vias 2 -> 1
- net SPI_DC: track 155.9 -> 179.0 mm, vias 2 -> 1
- net IO_INT: track 99.2 -> 121.9 mm, vias 1 -> 0
- net SPI_MOSI: track 166.7 -> 151.0 mm
- net SPI_SCK: track 155.6 -> 170.7 mm, vias 2 -> 1
- net MOT4A: track 81.1 -> 95.4 mm, vias 0 -> 4
- net FADER4_DIR: track 45.8 -> 59.2 mm, vias 1 -> 0
- net CS_EYE_R: track 119.4 -> 106.0 mm, vias 0 -> 1
- net CS_BELLY: track 96.2 -> 83.0 mm, vias 1 -> 0
- net FADER3_DIR: track 50.9 -> 40.7 mm, vias 1 -> 0
- net FADER2_WIPER: track 61.7 -> 71.7 mm
- net I2C_SCL: track 155.3 -> 164.8 mm, vias 2 -> 3
- net FADER3_PWM: track 49.8 -> 40.7 mm
- net DISP_RST: track 89.5 -> 80.7 mm, vias 1 -> 0
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Other:
- board text added: "3V3"
- board text added: "5V"
- board text added: "ARGB"
- board text added: "AUGEN"
- board text added: "BOOST"
- board text added: "BOOT"
- board text added: "CC1"
- board text added: "CC2"
- board text added: "DESK-MATE"
- board text added: "DIN"
- board text added: "DRV8833 · FADER 1+2"
- board text added: "DRV8833 · FADER 3+4"
- board text added: "ESP32-S3-DevKitC-1"
- board text added: "FRONTPANEL"
- board text added: "GND"
- board text added: "I2C · BME680"
- board text added: "IN+"
- board text added: "IN-"
- board text added: "JLCJLCJLCJLC"
- board text added: "Kabel vom Breakout"
- board text added: "Leon Fröhlich · 2026"
- board text added: "MAINBOARD · BASE"
- board text added: "MAINBOARD · BASE · Rev 1"
- board text added: "OUT+"
- board text added: "OUT-"
- board text added: "PAN"
- board text added: "RST"
- board text added: "Rev 1 · 2026-10"
- board text added: "SCL"
- board text added: "SDA"
- board text added: "SIG"
- board text added: "TILT"
- board text added: "USB-C IN 5V/3A"
- board text added: "VBUS"
- board text added: "VM 1-2: 5V 2-3: BOOST"
- board text removed: "Desk-Mate mainboard v1 2026-08"
