File: hardware/kicad/mainboard/mainboard.kicad_sch (KiCad schematic)
At the start: 50 parts, among them J1 USB-C 5V/3A (GCT USB4085), J10 Stepper 1A 1B 2A 2B, J2 IDC 2x15 -> Frontpanel, J3 Servo Pan (GND/5V/Sig), J4 Servo Tilt (GND/5V/Sig), J5 ARGB 5V/GND/Data, J6 BME680 (VCC GND SCL SDA SDO C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, J7 Augen-Kabel, J8 RST/BOOT extern, U1 ESP32-S3-DevKitC-1-N16R8, U2 LD1117V33, U3 DRV8833 Pololu #2130, U4 DRV8833 Pololu #2130 (Fader 3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, U5 MT3608 Boost ~9V (optional, 4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, U6 ESP32-C3 SuperMini Reserve, U7 A4988/TMC2209 Reserve

Commit message: Session 2026-10-03 00:27: Reserve raus (Stepper, C3, GPIO45, 7 Loetjumper), alle drei Platinen neu geroutet; Push und Falle 18 behoben
Parts:
- removed C8: 100u, Capacitor_THT:CP_Radial_D6.3mm_P2.50mm, symbol Device:C_Polarized
- removed J10: Stepper 1A 1B 2A 2B, Connector_PinHeader_2.54mm:PinHeader_1x04_P2.54mm_Vertical, symbol Connector_Generic:Conn_01x04
- removed JP2: C3 TX->S3 RX0, Jumper:SolderJumper-2_P1.3mm_Open_RoundedPad1.0x1.5mm, symbol Jumper:SolderJumper_2_Open
- removed JP3: S3 TX0->C3 RX, Jumper:SolderJumper-2_P1.3mm_Open_RoundedPad1.0x1.5mm, symbol Jumper:SolderJumper_2_Open
- removed JP4: VM: 1=5V 3=Boost, Jumper:SolderJumper-3_P1.3mm_Bridged12_RoundedPad1.0x1.5mm_NumberLabels, symbol Jumper:SolderJumper_3_Bridged12
- removed JP5: nSLEEP an 3V3, Jumper:SolderJumper-2_P1.3mm_Bridged_RoundedPad1.0x1.5mm, symbol Jumper:SolderJumper_2_Bridged
- removed JP6: STEP<-FADER3_PWM, Jumper:SolderJumper-2_P1.3mm_Open_RoundedPad1.0x1.5mm, symbol Jumper:SolderJumper_2_Open
- removed JP7: DIR<-FADER3_DIR, Jumper:SolderJumper-2_P1.3mm_Open_RoundedPad1.0x1.5mm, symbol Jumper:SolderJumper_2_Open
- removed JP8: EN<-FADER4_PWM, Jumper:SolderJumper-2_P1.3mm_Open_RoundedPad1.0x1.5mm, symbol Jumper:SolderJumper_2_Open
- removed U6: ESP32-C3 SuperMini Reserve, deskmate:ESP32-C3_SuperMini, symbol deskmate:ESP32-C3_SuperMini
- removed U7: A4988/TMC2209 Reserve, deskmate:A4988_Socket, symbol deskmate:A4988_Socket
- JP1: value BL45 (Strapping! offen lassen ausser Backlight-PWM) -> VM: 1=5V 3=Boost; footprint Jumper:SolderJumper-2_P1.3mm_Open_RoundedPad1.0x1.5mm -> Jumper:SolderJumper-3_P1.3mm_Bridged12_RoundedPad1.0x1.5mm_NumberLabels; symbol Jumper:SolderJumper_2_Open -> Jumper:SolderJumper_3_Bridged12
Connections:
- net DRV_SLEEP is gone; now on net 3V3: U3.7 (nSLEEP), U4.7 (nSLEEP)
- net 5V: now also JP1.1 (A)
- net GND: no longer J7.10 (Pin_10)
- net VBOOST: now also JP1.3 (B)
- net VM: now also JP1.2 (C)
- net BELLY_BL_PWM renamed DISP_RST
- net DISP_RST: now also J7.10 (Pin_10); no longer JP1.2 (B)
- net BL_PWM_45: no longer names the net of U1.37 (IO45)
- net BL_PWM_45: no longer JP1.1 (A)
- net UART0_RX: no longer names the net of U1.25 (RXD0/IO44)
- net UART0_TX: no longer names the net of U1.24 (TXD0/IO43)
- no-connect marks 40 -> 28
Other:
- note added: "MCU: ESP32-S3-DevKitC-1 gesteckt, USB-Ende zur Rueckwand, Antenne nach vorn ueber Kupfer-Sperrzone; DevKit-3V3 bleibt frei; 35-37 PSRAM, 19/20 USB, 43/44 UART0 frei, 0/3/45/46 Strapping"
- note added: "Motor: 2x DRV8833 (PWM+DIR), VM = 5V (JP1 Default) oder MT3608-Boost an U5; nSLEEP fest an 3V3"
- note removed: "MCU: ESP32-S3-DevKitC-1 gesteckt, USB-Ende zur Rueckwand, Antenne nach vorn ueber Kupfer-Sperrzone; DevKit-3V3 bleibt frei; 35-37 PSRAM, 19/20 USB, 0/3/46 Strapping"
- note removed: "Motor: 2x DRV8833 (PWM+DIR), VM = 5V (JP4 Default) oder MT3608-Boost an U5; nSLEEP ueber JP5 an 3V3"
- note removed: "Reserve (unbestueckt): A4988-Sockel an FADER3/4-Leitungen ueber Loetjumper; C3 SuperMini an UART0 ueber JP2/JP3"
- moved on the sheet: H1, H2, H3, H4, U5

Commit message: Session 2026-10-09 11:37: Platinen finalisiert: Teile von Reichelt, Silkscreen mit Logo und Pin-Namen, alle drei Boards neu geroutet
Parts:
- C1: value 1000u/10V -> 1000u/16V
- C11: footprint Capacitor_THT:CP_Radial_D5.0mm_P2.50mm -> Capacitor_THT:CP_Radial_D5.0mm_P2.00mm
- J1: value USB-C 5V/3A (GCT USB4085) -> USB-C-Breakout 5V/3A (VBUS GND CC1 CC2); footprint Connector_USB:USB_C_Receptacle_GCT_USB4085 -> TerminalBlock_Phoenix:TerminalBlock_Phoenix_MKDS-1,5-4-5.08_1x04_P5.08mm_Horizontal; symbol Connector:USB_C_Receptacle_USB2.0_16P -> Connector_Generic:Conn_01x04
- J3, J4, J5: footprint Connector_JST:JST_XH_B3B-XH-A_1x03_P2.50mm_Vertical -> Connector_PinHeader_2.54mm:PinHeader_1x03_P2.54mm_Vertical
- J6: value BME680 (VCC GND SCL SDA SDO CS) -> I2C / BME680 per Kabel; footprint Connector_PinSocket_2.54mm:PinSocket_1x06_P2.54mm_Vertical -> Connector_PinHeader_2.54mm:PinHeader_1x04_P2.54mm_Vertical; symbol Connector_Generic:Conn_01x06 -> Connector_Generic:Conn_01x04
- J7: value Augen-Kabel -> Augen-Kabel IDC 2x5; footprint Connector_PinHeader_2.54mm:PinHeader_1x10_P2.54mm_Vertical -> Connector_IDC:IDC-Header_2x05_P2.54mm_Vertical; symbol Connector_Generic:Conn_01x10 -> Connector_Generic:Conn_02x05_Odd_Even
- U1: value ESP32-S3-DevKitC-1-N16R8 -> ESP32-S3-DevKitC-1 (N16R8/N8R8)
Connections:
- net 3V3: no longer J7.2 (Pin_2)
- net CC1: now also J1.3 (Pin_3); no longer J1.A5 (CC1)
- net CC2: now also J1.4 (Pin_4); no longer J1.B5 (CC2)
- net GND: now also J1.2 (Pin_2), J7.2 (Pin_2), J7.6 (Pin_6); no longer J1.A1 (GND), J1.A12 (GND), J1.B1 (GND), J1.B12 (GND), J1.SH (SHIELD), J7.3 (Pin_3)
- net SPI_SCK: now also J7.3 (Pin_3); no longer J7.6 (Pin_6)
- net VBUS: now also J1.1 (Pin_1); no longer J1.A4 (VBUS), J1.A9 (VBUS), J1.B4 (VBUS), J1.B9 (VBUS)
- no-connect marks 28 -> 20
Other:
- note added: "Peripherie: Servos + ARGB als 1x3-Stiftleisten (470u, 330R + 1000u), I2C-Leiste fuer BME680, Augen-Kabel IDC 2x5, IDC zum Frontpanel"
- note added: "Versorgung: J1 (Schraubklemme <- USB-C-Breakout in der Rueckwand, CC1/CC2 je 5k1) 5V/3A -> Polyfuse -> SB540 -> 5V-Rail; LD1117V33 fuer Peripherie; PSU_SENSE vor der Diode (10k/15k -> 3,0 V)"
- note removed: "Peripherie: Servos (470u), ARGB (330R + 1000u), BME680-Sockel, Augen-Kabel, IDC zum Frontpanel"
- note removed: "Versorgung: J_PWR 5V/3A -> Polyfuse -> SB540 -> 5V-Rail; LD1117V33 fuer Peripherie; PSU_SENSE vor der Diode (10k/15k -> 3,0 V)"
- moved on the sheet: C1, C11, C2, C3, C4, C5, C6, C7, D1, F1, H1, H2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
